File: pcb-schematics/riscurino-1.0.sch (EAGLE design)
At the start: 49 parts, among them IC1 REG1117-3.3, IC2 REG1117-5.0, U1 ATXMEGA128A4U-AU, U2 MCP25625, U3 MCP25625, U4 CH340G, Y1 16MHz, Y2 12MHz, Y3 16MHz, Y4 16MHz

Commit message: Correct schematics and PCB uploaded.
Parts:
- C4: device rcl:CPOL-USC -> rcl:C-EUC0805
- U$1: value SWITCH_3X6 -> SWITCH_3X6_BIG; device riscurino:SWITCH_3X6 -> riscurino:SWITCH_3X6_BIG
- U2, U3: device MCP25625:MCP25625 -> MCP25625-fixed:MCP25625
Connections:
- net GND: now also C4.2; no longer C4.-
- net N$4: now also C4.1; no longer C4.+
- net VUSB: now also D2.A1
Other:
- note added: "1.0"
- note added: "16/oct/2017"
- note added: "Author: Ramiro Pareja (pareja@riscure.com)"
- note added: "CAN interfaces"
- note added: "Power supply, CPU and interfaces"
- note added: "Riscurino - Production ready"
